File: usbc-power.sch (KiCad schematic (older format))
At the start: 9 parts, among them J1 UJC-HP-3-SMT-TR, U1 NE555P

Commit message: modify pcb layout, add tracks and ground plane
Parts:
- C1, C2: footprint (none) -> Capacitor_THT:CP_Radial_D4.0mm_P1.50mm
- R1, R2, R3, R4: footprint (none) -> Resistor_THT:R_Axial_DIN0207_L6.3mm_D2.5mm_P2.54mm_Vertical
Changed lines of the file:
@@
 F 0 "R1" H 4918 2696 50  0000 L CNN
 F 1 "R" H 4918 2605 50  0000 L CNN
-F 2 "" H 4850 2650 50  0001 C CNN
+F 2 "Resistor_THT:R_Axial_DIN0207_L6.3mm_D2.5mm_P2.54mm_Vertical" H 4850 2650 50  0001 C CNN
 F 3 "~" H 4850 2650 50  0001 C CNN
 	1    4850 2650
@@
 F 0 "R2" H 4918 3446 50  0000 L CNN
 F 1 "R" H 4918 3355 50  0000 L CNN
-F 2 "" H 4850 3400 50  0001 C CNN
+F 2 "Resistor_THT:R_Axial_DIN0207_L6.3mm_D2.5mm_P2.54mm_Vertical" H 4850 3400 50  0001 C CNN
 F 3 "~" H 4850 3400 50  0001 C CNN
 	1    4850 3400
@@
 F 0 "R3" H 6468 2846 50  0000 L CNN
 F 1 "R" H 6468 2755 50  0000 L CNN
-F 2 "" H 6400 2800 50  0001 C CNN
+F 2 "Resistor_THT:R_Axial_DIN0207_L6.3mm_D2.5mm_P2.54mm_Vertical" H 6400 2800 50  0001 C CNN
 F 3 "~" H 6400 2800 50  0001 C CNN
 	1    6400 2800
@@
 F 0 "C2" H 5515 2596 50  0000 L CNN
 F 1 "CP1" H 5515 2505 50  0000 L CNN
-F 2 "" H 5400 2550 50  0001 C CNN
+F 2 "Capacitor_THT:CP_Radial_D4.0mm_P1.50mm" H 5400 2550 50  0001 C CNN
 F 3 "~" H 5400 2550 50  0001 C CNN
 	1    5400 2550
@@
 F 0 "C1" H 4965 4096 50  0000 L CNN
 F 1 "CP1" H 4965 4005 50  0000 L CNN
-F 2 "" H 4850 4050 50  0001 C CNN
+F 2 "Capacitor_THT:CP_Radial_D4.0mm_P1.50mm" H 4850 4050 50  0001 C CNN
 F 3 "~" H 4850 4050 50  0001 C CNN
 	1    4850 4050
@@
 F 0 "R4" H 7018 3496 50  0000 L CNN
 F 1 "R" H 7018 3405 50  0000 L CNN
-F 2 "" H 6950 3450 50  0001 C CNN
+F 2 "Resistor_THT:R_Axial_DIN0207_L6.3mm_D2.5mm_P2.54mm_Vertical" H 6950 3450 50  0001 C CNN
 F 3 "~" H 6950 3450 50  0001 C CNN
 	1    6950 3450

Commit message: add current limiting resistor, generate gerbers
Parts:
- added R5: R, Resistor_THT:R_Axial_DIN0207_L6.3mm_D2.5mm_P2.54mm_Vertical, symbol pspice:R
Connections:
- net GND: now also R5.1; no longer D1.1 (K)
- new net: D1.1 (K), R5.2
Changed lines of the file:
@@
 Wire Wire Line
 	6950 3700 7150 3700
-Text Label 7550 3700 0    50   ~ 0
-GND
 Wire Wire Line
 	7450 3700 7550 3700
+$Comp
+L pspice:R R5
+U 1 1 5F783173
+P 7800 3700
+F 0 "R5" V 7595 3700 50  0000 C CNN
+F 1 "R" V 7686 3700 50  0000 C CNN
+F 2 "Resistor_THT:R_Axial_DIN0207_L6.3mm_D2.5mm_P2.54mm_Vertical" H 7800 3700 50  0001 C CNN
+F 3 "~" H 7800 3700 50  0001 C CNN
+	1    7800 3700
+	0    1    1    0
+$EndComp
+Text Label 8050 3700 0    50   ~ 0
+GND
 $EndSCHEMATC
